Commit message: changed file path

File: urdf/drone.urdf (robot description, URDF)
Before this commit: robot drone, 9 links, 8 joints
Links:
- link base_link: geometry collision mesh filename=file://$(find drone)/meshes/base_link.STL; visual mesh filename=file://$(find drone)/meshes/base_link.STL
- link link_motor_front_left: geometry collision mesh filename=file://$(find drone)/meshes/link_motor_front_left.STL; visual mesh filename=file://$(find drone)/meshes/link_motor_front_left.STL
- link link_motor_front_right: geometry collision mesh filename=file://$(find drone)/meshes/link_motor_front_right.STL; visual mesh filename=file://$(find drone)/meshes/link_motor_front_right.STL
- link link_motor_rear_left: geometry collision mesh filename=file://$(find drone)/meshes/link_motor_rear_left.STL; visual mesh filename=file://$(find drone)/meshes/link_motor_rear_left.STL
- link link_motor_rear_right: geometry collision mesh filename=file://$(find drone)/meshes/link_motor_rear_right.STL; visual mesh filename=file://$(find drone)/meshes/link_motor_rear_right.STL
- link link_rotor_front_left: geometry collision mesh filename=file://$(find drone)/meshes/link_rotor_front_left.STL; visual mesh filename=file://$(find drone)/meshes/link_rotor_front_left.STL
- link link_rotor_front_right: geometry collision mesh filename=file://$(find drone)/meshes/link_rotor_front_right.STL; visual mesh filename=file://$(find drone)/meshes/link_rotor_front_right.STL
- link link_rotor_rear_left: geometry collision mesh filename=file://$(find drone)/meshes/link_rotor_rear_left.STL; visual mesh filename=file://$(find drone)/meshes/link_rotor_rear_left.STL
- link link_rotor_rear_right: geometry collision mesh filename=file://$(find drone)/meshes/link_rotor_rear_right.STL; visual mesh filename=file://$(find drone)/meshes/link_rotor_rear_right.STL
